File: makerspace-badge/makerspace-badge.kicad_pcb (KiCad board)
At the start: 2 copper layers, 66.1 x 53.3 mm, 83 parts, among them J1 Hexpansion-Connector, U1 ZD24C64A, U2 AW9523B, U3 AW9523B

Commit message: Maker Space badge, revision B
Parts:
- turned D1 to 125 degrees
- turned D10 to 0 degrees
- turned D11 to 180 degrees
- turned D12 to 180 degrees
- turned D13 to 0 degrees
- turned D14 to 180 degrees
- turned D15 to 180 degrees
- turned D16 to 0 degrees
- turned D17 to 145 degrees
- turned D18 to -70 degrees
- turned D19 to 70 degrees
- turned D2 to -30 degrees
- turned D20 to -145 degrees
- turned D21 to 0 degrees
- turned D22 to 180 degrees
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Connections:
- D1 pad 1: +3V3 -> /IO0_P0_7
- D1 pad 2: /IO0_P0_7 -> +3V3
- D10 pad 1: +3V3 -> /IO0_P1_7
- D10 pad 2: /IO0_P1_7 -> +3V3
- D11 pad 1: +3V3 -> /IO0_P0_6
- D11 pad 2: /IO0_P0_6 -> +3V3
- D12 pad 1: +3V3 -> /IO0_P0_6
- D12 pad 2: /IO0_P0_6 -> +3V3
- D13 pad 1: +3V3 -> /IO0_P0_6
- D13 pad 2: /IO0_P0_6 -> +3V3
- D14 pad 1: +3V3 -> /IO0_P0_5
- D14 pad 2: /IO0_P0_5 -> +3V3
- D15 pad 1: +3V3 -> /IO0_P0_5
- D15 pad 2: /IO0_P0_5 -> +3V3
- D16 pad 1: +3V3 -> /IO0_P0_5
- D16 pad 2: /IO0_P0_5 -> +3V3
- D17 pad 1: +3V3 -> /IO0_P0_4
- D17 pad 2: /IO0_P0_4 -> +3V3
- D18 pad 1: +3V3 -> /IO0_P0_4
- D18 pad 2: /IO0_P0_4 -> +3V3
- D19 pad 1: +3V3 -> /IO0_P0_3
- D19 pad 2: /IO0_P0_3 -> +3V3
- D2 pad 1: +3V3 -> /IO0_P1_4
- D2 pad 2: /IO0_P1_4 -> +3V3
- D20 pad 1: +3V3 -> /IO0_P0_3
- D20 pad 2: /IO0_P0_3 -> +3V3
- D21 pad 1: +3V3 -> /IO0_P0_2
- D21 pad 2: /IO0_P0_2 -> +3V3
- D22 pad 1: +3V3 -> /IO0_P0_2
- D22 pad 2: /IO0_P0_2 -> +3V3
- D23 pad 1: +3V3 -> /IO0_P0_1
- D23 pad 2: /IO0_P0_1 -> +3V3
- D24 pad 1: +3V3 -> /IO0_P0_1
- D24 pad 2: /IO0_P0_1 -> +3V3
- D25 pad 1: +3V3 -> /IO0_P0_0
- D25 pad 2: /IO0_P0_0 -> +3V3
- D26 pad 1: +3V3 -> /IO0_P0_0
- D26 pad 2: /IO0_P0_0 -> +3V3
- D27 pad 1: +3V3 -> /IO0_P0_0
- D27 pad 2: /IO0_P0_0 -> +3V3
- D28 pad 1: +3V3 -> /IO0_P1_3
- D28 pad 2: /IO0_P1_3 -> +3V3
- D29 pad 1: +3V3 -> /IO0_P1_3
- D29 pad 2: /IO0_P1_3 -> +3V3
- D3 pad 1: +3V3 -> /IO0_P1_4
- D3 pad 2: /IO0_P1_4 -> +3V3
- D30 pad 1: +3V3 -> /IO0_P1_2
- D30 pad 2: /IO0_P1_2 -> +3V3
- D31 pad 1: +3V3 -> /IO0_P1_2
- D31 pad 2: /IO0_P1_2 -> +3V3
- D32 pad 1: +3V3 -> /IO0_P1_1
- D32 pad 2: /IO0_P1_1 -> +3V3
- D33 pad 1: +3V3 -> /IO0_P1_1
- D33 pad 2: /IO0_P1_1 -> +3V3
- D34 pad 1: +3V3 -> /IO0_P1_0
- D34 pad 2: /IO0_P1_0 -> +3V3
- D35 pad 1: +3V3 -> /IO0_P1_0
- D35 pad 2: /IO0_P1_0 -> +3V3
- D36 pad 1: +3V3 -> /IO1_P0_7
- D36 pad 2: /IO1_P0_7 -> +3V3
- D37 pad 1: +3V3 -> /IO1_P0_7
- D37 pad 2: /IO1_P0_7 -> +3V3
- D38 pad 1: +3V3 -> /IO1_P1_4
- D38 pad 2: /IO1_P1_4 -> +3V3
- D39 pad 1: +3V3 -> /IO1_P1_4
- D39 pad 2: /IO1_P1_4 -> +3V3
- D4 pad 1: +3V3 -> /IO0_P1_5
- D4 pad 2: /IO0_P1_5 -> +3V3
- D40 pad 1: +3V3 -> /IO1_P0_6
- D40 pad 2: /IO1_P0_6 -> +3V3
- D41 pad 1: +3V3 -> /IO1_P0_6
- D41 pad 2: /IO1_P0_6 -> +3V3
- D42 pad 1: +3V3 -> /IO1_P0_6
- D42 pad 2: /IO1_P0_6 -> +3V3
- D43 pad 1: +3V3 -> /IO1_P0_5
- D43 pad 2: /IO1_P0_5 -> +3V3
- D44 pad 1: +3V3 -> /IO1_P0_5
- D44 pad 2: /IO1_P0_5 -> +3V3
- D45 pad 1: +3V3 -> /IO1_P0_4
- D45 pad 2: /IO1_P0_4 -> +3V3
- D46 pad 1: +3V3 -> /IO1_P0_4
- D46 pad 2: /IO1_P0_4 -> +3V3
- D47 pad 1: +3V3 -> /IO1_P0_3
- D47 pad 2: /IO1_P0_3 -> +3V3
- D48 pad 1: +3V3 -> /IO1_P0_3
- D48 pad 2: /IO1_P0_3 -> +3V3
- D49 pad 1: +3V3 -> /IO1_P0_2
- D49 pad 2: /IO1_P0_2 -> +3V3
- D5 pad 1: +3V3 -> /IO0_P1_5
- D5 pad 2: /IO0_P1_5 -> +3V3
- D50 pad 1: +3V3 -> /IO1_P0_2
- D50 pad 2: /IO1_P0_2 -> +3V3
- D51 pad 1: +3V3 -> /IO1_P0_1
- D51 pad 2: /IO1_P0_1 -> +3V3
- D52 pad 1: +3V3 -> /IO1_P0_1
- D52 pad 2: /IO1_P0_1 -> +3V3
- D53 pad 1: +3V3 -> /IO1_P0_1
- D53 pad 2: /IO1_P0_1 -> +3V3
- D54 pad 1: +3V3 -> /IO1_P0_0
- D54 pad 2: /IO1_P0_0 -> +3V3
- D55 pad 1: +3V3 -> /IO1_P0_0
- D55 pad 2: /IO1_P0_0 -> +3V3
- D56 pad 1: +3V3 -> /IO1_P0_0
- D56 pad 2: /IO1_P0_0 -> +3V3
- D57 pad 1: +3V3 -> /IO1_P1_0
- D57 pad 2: /IO1_P1_0 -> +3V3
- D58 pad 1: +3V3 -> /IO1_P1_0
- D58 pad 2: /IO1_P1_0 -> +3V3
- D59 pad 1: +3V3 -> /IO1_P1_0
- D59 pad 2: /IO1_P1_0 -> +3V3
- D6 pad 1: +3V3 -> /IO0_P1_6
- D6 pad 2: /IO0_P1_6 -> +3V3
- D60 pad 1: +3V3 -> /IO1_P1_1
- D60 pad 2: /IO1_P1_1 -> +3V3
- D61 pad 1: +3V3 -> /IO1_P1_1
- D61 pad 2: /IO1_P1_1 -> +3V3
- D62 pad 1: +3V3 -> /IO1_P1_2
- D62 pad 2: /IO1_P1_2 -> +3V3
- D63 pad 1: +3V3 -> /IO1_P1_2
- D63 pad 2: /IO1_P1_2 -> +3V3
- D64 pad 1: +3V3 -> /IO1_P1_3
- D64 pad 2: /IO1_P1_3 -> +3V3
- D65 pad 1: +3V3 -> /IO1_P1_3
- D65 pad 2: /IO1_P1_3 -> +3V3
- D66 pad 1: +3V3 -> /IO0_P0_7
- D66 pad 2: /IO0_P0_7 -> +3V3
- D7 pad 1: +3V3 -> /IO0_P1_6
- D7 pad 2: /IO0_P1_6 -> +3V3
- D8 pad 1: +3V3 -> /IO0_P1_7
- D8 pad 2: /IO0_P1_7 -> +3V3
- D9 pad 1: +3V3 -> /IO0_P1_7
- D9 pad 2: /IO0_P1_7 -> +3V3
